File: schematics/dev_v1/usb_dip_v1.sch (EAGLE design)
At the start: 41 parts, among them U1 PRTR5V0U2X, U2 PRTR5V0U2X, U3 PRTR5V0U2X, U4 PRTR5V0U2X, U5 PRTR5V0U2X

Commit message: osh order
Parts:
- removed R2: ?, rcl:R-EU_R0805
- added Q1: (no value), adafruit:CRYSTALSM49
- U$10: value (none) -> USB-PWR; device adafruit:CERMOSCILL-THM -> adafruit:USB-PWR
Connections:
- removed net N$23: R2.1, U$1.OVCJ
- new net V_UP: U$1.VBUSM, U$8.VBUS
- net GND: now also U$1.TESTJ
- net N$27: now also Q1.2; no longer U$10.IN
- net N$28: now also Q1.1; no longer U$10.OUT
- net VCC: now also U$1.OVCJ, U$1.PWRJ, U$10.VBUS; no longer R2.2
Changed lines of the file:
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@@
 <part name="GND12" library="supply1" deviceset="GND" device=""/>
 <part name="R1" library="rcl" deviceset="R-EU_" device="R0805" value="2.7k"/>
-<part name="R2" library="rcl" deviceset="R-EU_" device="R0805" value="?"/>
 <part name="R3" library="rcl" deviceset="R-EU_" device="R0805" value="10k"/>
 <part name="R4" library="rcl" deviceset="R-EU_" device="R0805" value="10k"/>
@@
 <part name="GND13" library="supply1" deviceset="GND" device=""/>
 <part name="P+6" library="supply1" deviceset="VCC" device=""/>
-<part name="U$10" library="adafruit" deviceset="CERMOSCILL" device="-THM"/>
-<part name="GND14" library="supply1" deviceset="GND" device=""/>
 <part name="P+7" library="supply1" deviceset="VCC" device=""/>
 <part name="LED1" library="led" deviceset="LED" device="CHIP-LED0805"/>
@@
 <part name="GND17" library="supply1" deviceset="GND" device=""/>
 <part name="P+2" library="supply1" deviceset="VCC" device=""/>
+<part name="GND18" library="supply1" deviceset="GND" device=""/>
+<part name="Q1" library="adafruit" deviceset="CRYSTAL" device="SM49"/>
+<part name="U$10" library="adafruit" deviceset="USB-PWR" device=""/>
+<part name="GND14" library="supply1" deviceset="GND" device=""/>
 </parts>
 <sheets>
@@
 <instance part="GND12" gate="1" x="139.7" y="116.84"/>
 <instance part="R1" gate="G$1" x="111.76" y="177.8"/>
-<instance part="R2" gate="G$1" x="109.22" y="193.04" rot="R180"/>
 <instance part="R3" gate="G$1" x="83.82" y="190.5" rot="R270"/>
 <instance part="R4" gate="G$1" x="76.2" y="190.5" rot="R270"/>
@@
 <instance part="GND13" gate="1" x="111.76" y="208.28"/>
 <instance part="P+6" gate="VCC" x="116.84" y="220.98"/>
-<instance part="U$10" gate="G$1" x="93.98" y="208.28" rot="R270"/>
-<instance part="GND14" gate="1" x="88.9" y="203.2"/>
-<instance part="P+7" gate="VCC" x="96.52" y="198.12"/>
+<instance part="P+7" gate="VCC" x="116.84" y="198.12"/>
 <instance part="LED1" gate="G$1" x="180.34" y="236.22" rot="R180"/>
 <instance part="LED2" gate="G$1" x="190.5" y="238.76"/>
@@
 <instance part="GND17" gate="1" x="88.9" y="78.74"/>
 <instance part="P+2" gate="VCC" x="58.42" y="93.98"/>
+<instance part="GND18" gate="1" x="111.76" y="190.5"/>
+<instance part="Q1" gate="G$1" x="99.06" y="208.28" rot="R90"/>
+<instance part="U$10" gate="G$1" x="86.36" y="17.78"/>
+<instance part="GND14" gate="1" x="106.68" y="7.62"/>
 </instances>
 <busses>
@@
 <wire x1="121.92" y1="213.36" x2="111.76" y2="213.36" width="0.1524" layer="91"/>
 <wire x1="111.76" y1="213.36" x2="111.76" y2="210.82" width="0.1524" layer="91"/>
-</segment>
-<segment>
-<pinref part="U$10" gate="G$1" pin="GND"/>
-<wire x1="91.44" y1="208.28" x2="88.9" y2="208.28" width="0.1524" layer="91"/>
-<wire x1="88.9" y1="208.28" x2="88.9" y2="205.74" width="0.1524" layer="91"/>
-<pinref part="GND14" gate="1" pin="GND"/>
 </segment>
 <segment>
@@
 <pinref part="GND17" gate="1" pin="GND"/>
 <wire x1="88.9" y1="86.36" x2="88.9" y2="81.28" width="0.1524" layer="91"/>
+</segment>
+<segment>
+<pinref part="U$1" gate="G$1" pin="TESTJ"/>
+<wire x1="121.92" y1="198.12" x2="119.38" y2="198.12" width="0.1524" layer="91"/>
+<wire x1="119.38" y1="198.12" x2="119.38" y2="200.66" width="0.1524" layer="91"/>
+<wire x1="119.38" y1="200.66" x2="111.76" y2="200.66" width="0.1524" layer="91"/>
+<wire x1="111.76" y1="200.66" x2="111.76" y2="193.04" width="0.1524" layer="91"/>
+<pinref part="GND18" gate="1" pin="GND"/>
+</segment>
+<segment>
+<pinref part="U$10" gate="G$1" pin="GND"/>
+<pinref part="GND14" gate="1" pin="GND"/>
+<wire x1="99.06" y1="12.7" x2="106.68" y2="12.7" width="0.1524" layer="91"/>
+<wire x1="106.68" y1="12.7" x2="106.68" y2="10.16" width="0.1524" layer="91"/>
 </segment>
 </net>
@@
 </segment>
 <segment>
-<pinref part="R2" gate="G$1" pin="2"/>
 <pinref part="P+7" gate="VCC" pin="VCC"/>
-<wire x1="104.14" y1="193.04" x2="96.52" y2="193.04" width="0.1524" layer="91"/>
-<wire x1="96.52" y1="193.04" x2="96.52" y2="195.58" width="0.1524" layer="91"/>
+<pinref part="U$1" gate="G$1" pin="PWRJ"/>
+<pinref part="U$1" gate="G$1" pin="OVCJ"/>
+<wire x1="116.84" y1="195.58" x2="121.92" y2="195.58" width="0.1524" layer="91"/>
+<wire x1="121.92" y1="193.04" x2="116.84" y2="193.04" width="0.1524" layer="91"/>
+<wire x1="116.84" y1="193.04" x2="116.84" y2="195.58" width="0.1524" layer="91"/>
+<junction x="116.84" y="195.58"/>
 </segment>
 <segment>
@@
 <wire x1="58.42" y1="86.36" x2="60.96" y2="86.36" width="0.1524" layer="91"/>
 </segment>
+<segment>
+<pinref part="U$10" gate="G$1" pin="VBUS"/>
+<wire x1="99.06" y1="22.86" x2="111.76" y2="22.86" width="0.1524" layer="91"/>
+<label x="101.6" y="22.86" size="1.778" layer="95"/>
+</segment>
 </net>
 <net name="DM1" class="0">
@@
 </segment>
 </net>
-<net name="N$23" class="0">
-<segment>
-<pinref part="U$1" gate="G$1" pin="OVCJ"/>
-<pinref part="R2" gate="G$1" pin="1"/>
-<wire x1="114.3" y1="193.04" x2="116.84" y2="193.04" width="0.1524" layer="91"/>
-<wire x1="116.84" y1="193.04" x2="116.84" y2="195.58" width="0.1524" layer="91"/>
-<wire x1="116.84" y1="195.58" x2="121.92" y2="195.58" width="0.1524" layer="91"/>
-</segment>
-</net>
 <net name="N$24" class="0">
 <segment>
@@
 <net name="N$27" class="0">
 <segment>
-<pinref part="U$10" gate="G$1" pin="IN"/>
-<wire x1="99.06" y1="213.36" x2="99.06" y2="215.9" width="0.1524" layer="91"/>
-<wire x1="99.06" y1="215.9" x2="104.14" y2="215.9" width="0.1524" layer="91"/>
-<wire x1="104.14" y1="215.9" x2="104.14" y2="205.74" width="0.1524" layer="91"/>
+<wire x1="99.06" y1="210.82" x2="99.06" y2="213.36" width="0.1524" layer="91"/>
+<wire x1="99.06" y1="213.36" x2="104.14" y2="213.36" width="0.1524" layer="91"/>
+<wire x1="104.14" y1="213.36" x2="104.14" y2="205.74" width="0.1524" layer="91"/>
 <pinref part="U$1" gate="G$1" pin="XOUT"/>
 <wire x1="104.14" y1="205.74" x2="121.92" y2="205.74" width="0.1524" layer="91"/>
+<pinref part="Q1" gate="G$1" pin="2"/>
 </segment>
 </net>
@@
 <segment>
 <pinref part="U$1" gate="G$1" pin="XIN"/>
-<wire x1="121.92" y1="203.2" x2="104.14" y2="203.2" width="0.1524" layer="91"/>
-<wire x1="104.14" y1="203.2" x2="104.14" y2="200.66" width="0.1524" layer="91"/>
-<pinref part="U$10" gate="G$1" pin="OUT"/>
-<wire x1="104.14" y1="200.66" x2="99.06" y2="200.66" width="0.1524" layer="91"/>
-<wire x1="99.06" y1="200.66" x2="99.06" y2="203.2" width="0.1524" layer="91"/>
+<wire x1="121.92" y1="203.2" x2="99.06" y2="203.2" width="0.1524" layer="91"/>
+<wire x1="99.06" y1="203.2" x2="99.06" y2="205.74" width="0.1524" layer="91"/>
+<pinref part="Q1" gate="G$1" pin="1"/>
 </segment>
 </net>
@@
 </segment>
 </net>
+<net name="V_UP" class="0">
+<segment>
+<pinref part="U$8" gate="G$1" pin="VBUS"/>
+<wire x1="127" y1="129.54" x2="127" y2="142.24" width="0.1524" layer="91"/>
+<wire x1="127" y1="142.24" x2="137.16" y2="142.24" width="0.1524" layer="91"/>
+<label x="129.54" y="142.24" size="1.778" layer="95"/>
+</segment>
+<segment>
+<pinref part="U$1" gate="G$1" pin="VBUSM"/>
+<wire x1="121.92" y1="185.42" x2="99.06" y2="185.42" width="0.1524" layer="91"/>
+<label x="99.06" y="185.42" size="1.778" layer="95"/>
+</segment>
+</net>
