File: schematics/v3/queso_dip_v3.sch (EAGLE design)
At the start: 43 parts, among them Q1 FOXSDLF/120-20, U1 PRTR5V0U2X,215, U2 PRTR5V0U2X,215, U3 PRTR5V0U2X,215, U4 PRTR5V0U2X,215, U5 PRTR5V0U2X,215, X1 USB-A-HU, X2 USB-A-HU, X3 USB-A-HU, X4 USB-A-HU

Commit message: routing for version3
Parts:
- removed U$10: USB-PWR, adafruit:USB-PWR
- added C7: 100nF, rcl:C-EUC0805
Connections:
- net GND: now also C7.1; no longer U$10.GND
- net VCC: now also C7.2; no longer U$10.VBUS
Changed lines of the file:
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@@
 <part name="GND18" library="supply1" deviceset="GND" device=""/>
 <part name="Q1" library="adafruit" deviceset="CRYSTAL" device="SM49" value="FOXSDLF/120-20"/>
-<part name="U$10" library="adafruit" deviceset="USB-PWR" device=""/>
-<part name="GND14" library="supply1" deviceset="GND" device=""/>
 <part name="X1" library="con-usb" deviceset="USB" device="-A-HU"/>
 <part name="X2" library="con-usb" deviceset="USB" device="-A-HU"/>
@@
 <part name="GND20" library="supply1" deviceset="GND" device=""/>
 <part name="SJ2" library="SparkFun-Retired" deviceset="SOLDERJUMPER_2WAY" device="T"/>
+<part name="C7" library="rcl" deviceset="C-EU" device="C0805" value="100nF"/>
+<part name="P+10" library="supply1" deviceset="VCC" device=""/>
+<part name="GND21" library="supply1" deviceset="GND" device=""/>
 </parts>
 <sheets>
@@
 <instance part="GND18" gate="1" x="111.76" y="190.5"/>
 <instance part="Q1" gate="G$1" x="99.06" y="208.28" rot="R90"/>
-<instance part="U$10" gate="G$1" x="86.36" y="17.78"/>
-<instance part="GND14" gate="1" x="106.68" y="7.62"/>
 <instance part="X1" gate="G$1" x="236.22" y="127"/>
 <instance part="X2" gate="G$1" x="236.22" y="144.78"/>
@@
 <instance part="GND20" gate="1" x="124.46" y="297.18"/>
 <instance part="SJ2" gate="G$1" x="63.5" y="248.92" rot="R270"/>
+<instance part="C7" gate="G$1" x="134.62" y="223.52" rot="R180"/>
+<instance part="P+10" gate="VCC" x="134.62" y="231.14"/>
+<instance part="GND21" gate="1" x="134.62" y="218.44"/>
 </instances>
 <busses>
@@
 </segment>
 <segment>
-<pinref part="U$10" gate="G$1" pin="GND"/>
-<pinref part="GND14" gate="1" pin="GND"/>
-<wire x1="99.06" y1="12.7" x2="106.68" y2="12.7" width="0.1524" layer="91"/>
-<wire x1="106.68" y1="12.7" x2="106.68" y2="10.16" width="0.1524" layer="91"/>
-</segment>
-<segment>
 <pinref part="U$3" gate="G$1" pin="GNDOUT"/>
 <wire x1="139.7" y1="304.8" x2="139.7" y2="302.26" width="0.1524" layer="91"/>
@@
 <wire x1="124.46" y1="302.26" x2="124.46" y2="299.72" width="0.1524" layer="91"/>
 <pinref part="GND20" gate="1" pin="GND"/>
+</segment>
+<segment>
+<pinref part="C7" gate="G$1" pin="1"/>
+<pinref part="GND21" gate="1" pin="GND"/>
 </segment>
 </net>
@@
 </segment>
 <segment>
-<pinref part="U$10" gate="G$1" pin="VBUS"/>
-<wire x1="99.06" y1="22.86" x2="111.76" y2="22.86" width="0.1524" layer="91"/>
-<label x="101.6" y="22.86" size="1.778" layer="95"/>
-</segment>
-</net>
+<pinref part="C7" gate="G$1" pin="2"/>
+<pinref part="P+10" gate="VCC" pin="VCC"/>
+</segment>
+</net>
