File: schematics/v2/queso_dip_v2.brd (EAGLE design)
At the start: 41 x 50 mm, 43 parts, among them U1 PRTR5V0U2X, U2 PRTR5V0U2X, U3 PRTR5V0U2X, U4 PRTR5V0U2X, U5 PRTR5V0U2X

Commit message: added new version
Parts:
- removed R2: ?, rcl:R0805
- added Q1: FOXSDLF/120-20, adafruit:SM49
- C1, C2, C3, C4, C5, C6: value 10uF -> VJ1210V106ZXJTW1BC
- F1, F2, F3, F4: value (none) -> PTS12066V110
- LED1, LED2, LED3, LED4, LED5: value (none) -> 150080BS75000
- R5, R6, R7: value 330R -> ERJ-6ENF3300V
- U$10: value (none) -> USB-PWR; device adafruit:CERM_OSC -> adafruit:USB-MINIB-THM-MOLEX-PWRONLY
- U$3, U$4, U$6, U$7: value USB_TYPE_A_FEMALE_TH -> amp 787616-1
- U$8: value USB-MINIB-5PIN -> 10118194-0001LF
- U1, U2, U3, U4, U5: value PRTR5V0U2X -> PRTR5V0U2X,215
- moved U$10 22.6 mm to (12.1, 3.50), turned to 0 degrees
- moved U5 14.9 mm to (10.2, 25.0)
- moved C6 12.8 mm to (18.0, 30.3), turned to 270 degrees
- moved F4 6.70 mm to (27.2, 10.1), turned to 270 degrees
- moved C5 6.38 mm to (23.7, 29.4), turned to 180 degrees
- moved C1 5.02 mm to (21.1, 10.6), flipped to the top, turned to 0 degrees
- moved LED4 4.00 mm to (14.0, 36.5)
- moved LED5 4.00 mm to (11.5, 36.5)
- moved R6 3.86 mm to (16.3, 35.9)
- moved C3 3.13 mm to (24.2, 24.4)
- moved F1 3.06 mm to (27.4, 24.4), flipped to the bottom
- moved JP1 1.90 mm to (10.8, 11.5)
- moved R5 1.30 mm to (18.5, 36.6)
- moved PAD1 1.00 mm to (8.50, 3.00)
- moved PAD2 1.00 mm to (13.5, 3.00)
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Connections:
- removed net N$23: R2.1, U$1.26
- new net V_UP: U$1.18, U$8.VBUS
- net GND: now also U$1.27, U$10.GND; no longer U$10.P$2
- net N$27: now also Q1.2; no longer U$10.P$1
- net N$28: now also Q1.1; no longer U$10.P$3
- net VCC: now also U$1.25, U$1.26, U$10.VBUS; no longer R2.2
Routing:
- net V_UP: track 0.00 -> 19.8 mm, vias 0 -> 1
- net GND: track 398.2 -> 412.1 mm, vias 10 -> 7
- net VCC: track 152.2 -> 165.7 mm, vias 11 -> 9
- net N$18: track 39.7 -> 30.7 mm
- net N$23: track 8.09 -> 0.00 mm
- net N$32: track 23.7 -> 17.8 mm
- net N$28: track 8.02 -> 13.9 mm, vias 0 -> 1
- net DP3: track 23.6 -> 28.2 mm
- net DM3: track 23.6 -> 27.9 mm
- net DM1: track 29.5 -> 32.9 mm
- net DMU: track 31.4 -> 34.5 mm, vias 1 -> 2
- net DPU: track 31.4 -> 34.4 mm, vias 1 -> 2
- net N$12: track 3.58 -> 6.13 mm
- net N$30: track 6.50 -> 3.97 mm, vias 0 -> 1
- net N$15: track 9.28 -> 7.63 mm
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Other:
- board text added: "JKW v0.2"
- board text added: "QUESO DIP"
- board text removed: "SALSA DIP"

Commit message: added order notes to all boards
Other:
- board text added: "never ordered"
Changed lines of the file:
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@@
 <wire x1="16" y1="0.8" x2="6" y2="0.8" width="0.6096" layer="21"/>
 <wire x1="6" y1="0.8" x2="6" y2="7.5" width="0.6096" layer="21"/>
+<text x="-4" y="18.4" size="1.778" layer="21" rot="R90">never ordered</text>
 </plain>
 <attributes>
