File: schematics/v5/queso_dip_v5.brd (EAGLE design)
At the start: 41 x 50 mm, 43 parts, among them K1 61400826021, K2 61400826021, Q1 FOXSDLF/120-20, U1 PRTR5V0U2X,215, U2 PRTR5V0U2X,215, U3 PRTR5V0U2X,215, U4 PRTR5V0U2X,215, U5 PRTR5V0U2X,215

Commit message: added order notes to all boards
Parts:
- moved SJ2 0.20 mm to (9.10, 44.6)
Routing:
- net DP2: track 17.2 -> 22.4 mm
- net DP4: track 23.8 -> 28.3 mm
- net DM1: track 22.3 -> 26.7 mm
- net DM4: track 24.1 -> 28.3 mm
- net DM3: track 16.1 -> 19.6 mm
- net DP3: track 17.0 -> 19.4 mm
- net DP1: track 24.6 -> 26.6 mm
- net CHR_IN: track 6.71 -> 7.23 mm
Other:
- board text added: "dual double jacks not ordered"
