File: schematics/v4/queso_dip_v4.brd (EAGLE design)
At the start: 41 x 50 mm, 45 parts, among them Q1 FOXSDLF/120-20, U1 PRTR5V0U2X,215, U2 PRTR5V0U2X,215, U3 PRTR5V0U2X,215, U4 PRTR5V0U2X,215, U5 PRTR5V0U2X,215, X1 USB-A-HU, X2 USB-A-HU, X3 USB-A-HU, X4 USB-A-HU

Commit message: added order notes to all boards
Other:
- board text added: "fixed LEDs, never ordered"
Changed lines of the file:
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@@
 <text x="24.4" y="27.2" size="1.27" layer="25">A  4  3  2  1</text>
 <circle x="4" y="31.9" radius="1.204159375" width="0.254" layer="26"/>
+<text x="-3.1" y="10.7" size="1.778" layer="23" rot="R90">fixed LEDs, never ordered</text>
 </plain>
 <attributes>
@@
 <wire x1="19.0507" y1="42.4501" x2="19.2" y2="42.3008" width="0.254" layer="1"/>
 <wire x1="19.2" y1="42.3008" x2="19.2" y2="39.7" width="0.254" layer="1"/>
-<wire x1="33.2" y1="20.5" x2="33.3" y2="23.5" width="0" layer="19" extent="1-1"/>
-<wire x1="17.7" y1="3.7" x2="17.62" y2="3.3" width="0" layer="19" extent="1-1"/>
-<wire x1="11.8" y1="15.7" x2="11.5" y2="17.2" width="0" layer="19" extent="16-16"/>
 </signal>
 <signal name="INT0">

Commit message: fixed micro usb
Parts:
- removed U$8: 10118194-0001LF, SparkFun-Connectors:USB-MINIB
- added JP2: USB-RECEPTABLE, daspilker:FCI-10103594-0001LF
- moved SJ2 1.30 mm to (9.80, 45.8), turned to 90 degrees
Connections:
- net DMU: now also JP2.2; no longer U$8.D-
- net DPU: now also JP2.3; no longer U$8.D+
- net GND: now also JP2.5; no longer U$8.GND, U$8.MTN1, U$8.MTN2, U$8.MTN3, U$8.MTN4
- net V_UP: now also JP2.1; no longer U$8.VBUS
Routing:
- net GND: track 296.8 -> 276.2 mm, vias 13 -> 14
- net DPU: track 22.9 -> 25.7 mm
- net DMU: track 30.0 -> 32.8 mm
- net V_UP: track 20.6 -> 23.3 mm
- net CHR_IN: track 6.71 -> 8.75 mm
- net VOUT2: track 13.8 -> 12.7 mm
