File: schematics/v4_ordered/queso_dip_v4_3.brd (EAGLE design)
At the start: 41 x 50 mm, 46 parts, among them Q1 FOXSDLF/120-20, U1 PRTR5V0U2X,215, U2 PRTR5V0U2X,215, U3 PRTR5V0U2X,215, U4 PRTR5V0U2X,215, U5 PRTR5V0U2X,215, X1 USB-A-HU, X2 USB-A-HU, X3 USB-A-HU, X4 USB-A-HU

Commit message: ordered v4 with correct vss
Parts:
- moved R1 1.90 mm to (13.0, 21.7), turned to 270 degrees
Connections:
- net GND: now also R1.1
- net N$18: no longer R1.1
Routing:
- net N$18: track 30.9 -> 23.4 mm
- net GND: track 288.1 -> 291.1 mm
- net VIN: track 52.0 -> 53.9 mm
- net N$22: track 6.55 -> 7.53 mm
Other:
- board text added: "JKW v0.43"
- board text added: "ordered 2016/03/16 elecrow"
- board text removed: "JKW v0.42"
- board text removed: "fixed LEDs, never ordered"
