File: schematics/v4_ordered/queso_dip_v4_3.sch (EAGLE design)
At the start: 46 parts, among them Q1 FOXSDLF/120-20, U1 PRTR5V0U2X,215, U2 PRTR5V0U2X,215, U3 PRTR5V0U2X,215, U4 PRTR5V0U2X,215, U5 PRTR5V0U2X,215, X1 USB-A-HU, X2 USB-A-HU, X3 USB-A-HU, X4 USB-A-HU

Commit message: ordered v4 with correct vss
Connections:
- net GND: now also R1.1
- net N$18: no longer R1.1
Changed lines of the file:
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@@
 <part name="U$2" library="logo" deviceset="LOGO_3X3_COPPER" device=""/>
 <part name="U$5" library="logo" deviceset="LOGO_10X10_SILK" device=""/>
+<part name="GND12" library="supply1" deviceset="GND" device=""/>
 </parts>
 <sheets>
@@
 <instance part="U$2" gate="G$1" x="5.08" y="2.54"/>
 <instance part="U$5" gate="G$1" x="177.8" y="2.54"/>
+<instance part="GND12" gate="1" x="43.18" y="149.86"/>
 </instances>
 <busses>
@@
 <pinref part="C7" gate="G$1" pin="1"/>
 <pinref part="GND21" gate="1" pin="GND"/>
+</segment>
+<segment>
+<pinref part="R1" gate="G$1" pin="1"/>
+<wire x1="66.04" y1="175.26" x2="43.18" y2="175.26" width="0.1524" layer="91"/>
+<pinref part="GND12" gate="1" pin="GND"/>
+<wire x1="43.18" y1="175.26" x2="43.18" y2="152.4" width="0.1524" layer="91"/>
 </segment>
 </net>
@@
 <wire x1="66.04" y1="167.64" x2="66.04" y2="170.18" width="0.1524" layer="91"/>
 <junction x="66.04" y="170.18"/>
-<pinref part="R1" gate="G$1" pin="1"/>
-<wire x1="66.04" y1="175.26" x2="53.34" y2="175.26" width="0.1524" layer="91"/>
-<wire x1="53.34" y1="175.26" x2="53.34" y2="170.18" width="0.1524" layer="91"/>
-<junction x="53.34" y="170.18"/>
-</segment>
-</net>
+</segment>
+</net>
