File: schematics/v4_ordered/queso_dip_v4_4.brd (EAGLE design)
At the start: 41 x 50 mm, 46 parts, among them Q1 FOXSDLF/120-20, U1 PRTR5V0U2X,215, U2 PRTR5V0U2X,215, U3 PRTR5V0U2X,215, U4 PRTR5V0U2X,215, U5 PRTR5V0U2X,215, X1 USB-A-HU, X2 USB-A-HU, X3 USB-A-HU, X4 USB-A-HU

Commit message: updated v4.4
Routing:
- net GND: track 289.9 -> 283.5 mm
Other:
- board text added: "JKW v0.44"
- board text removed: "JKW v0.43"
Changed lines of the file:
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@@
 DIP </text>
 <text x="5.7049" y="49.2006" size="1.27" layer="22" font="vector" ratio="12" rot="MR0" align="top-left"> JKW
-v0.43</text>
+v0.44</text>
 <wire x1="34" y1="50" x2="24" y2="50" width="0.6096" layer="21"/>
 <wire x1="24" y1="50" x2="24" y2="42.3" width="0.6096" layer="21"/>
@@
 <wire x1="25.4" y1="10.2" x2="25.4" y2="3.8" width="0.254" layer="1"/>
 <wire x1="25.4" y1="3.8" x2="25.5" y2="3.7" width="0.254" layer="1"/>
-<wire x1="24.3593" y1="25.6593" x2="25" y2="26.3" width="0.254" layer="16"/>
-<wire x1="25" y1="26.3" x2="28.706" y2="26.3" width="0.254" layer="16"/>
-<wire x1="28.706" y1="26.3" x2="30.02" y2="24.986" width="0.254" layer="16"/>
 <via x="18.2" y="31.9" extent="1-16" drill="0.6"/>
 <wire x1="18.4" y1="31.2" x2="18.4" y2="30.1" width="0.254" layer="1"/>
@@
 <wire x1="13" y1="22.65" x2="13" y2="23.464" width="0.254" layer="16"/>
 <wire x1="13" y1="23.464" x2="11.478" y2="24.986" width="0.254" layer="16"/>
-<wire x1="33.2" y1="20.5" x2="33.3" y2="23.5" width="0" layer="19" extent="1-1"/>
-<wire x1="17.7" y1="3.7" x2="17.62" y2="3.3" width="0" layer="19" extent="1-1"/>
-<wire x1="11.8" y1="15.7" x2="11.5" y2="17.2" width="0" layer="19" extent="16-16"/>
 </signal>
 <signal name="INT0">
