File: schematics/v5_double_dual/queso_dip_v5.brd (EAGLE design)
At the start: 41 x 50 mm, 43 parts, among them K1 61400826021, K2 61400826021, Q1 FOXSDLF/120-20, U1 PRTR5V0U2X,215, U2 PRTR5V0U2X,215, U3 PRTR5V0U2X,215, U4 PRTR5V0U2X,215, U5 PRTR5V0U2X,215

Commit message: ordered v4 with correct vss
Connections:
- net GND: now also R1.1
- net N$18: no longer R1.1
Changed lines of the file:
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@@
 <wire x1="25.8" y1="11.4" x2="26.6" y2="11.4" width="0.254" layer="16"/>
 <via x="26.6" y="11.4" extent="1-16" drill="0.6"/>
-<wire x1="26.6" y1="11.4" x2="25.4" y2="10.2" width="0" layer="19" extent="1-16"/>
-<wire x1="25.4" y1="10.2" x2="25.4" y2="3.8" width="0" layer="19" extent="1-16"/>
-<wire x1="25.4" y1="3.8" x2="25.5" y2="3.7" width="0" layer="19" extent="1-16"/>
 <wire x1="24.3593" y1="24.5031" x2="24.3593" y2="25.6593" width="0.254" layer="16"/>
 <wire x1="24.3593" y1="25.6593" x2="25" y2="26.3" width="0.254" layer="16"/>
@@
 <wire x1="22.3" y1="4.9" x2="17.6" y2="4.9" width="0.254" layer="1"/>
 <wire x1="17.6" y1="4.9" x2="16.6" y2="3.9" width="0.254" layer="1"/>
+<contactref element="R1" pad="1"/>
 <wire x1="33.2" y1="20.5" x2="33.3" y2="23.5" width="0" layer="19" extent="1-1"/>
-<wire x1="25.4" y1="3.8" x2="24.2" y2="3" width="0" layer="19" extent="1-1"/>
 <wire x1="11.8" y1="15.7" x2="11.5" y2="17.2" width="0" layer="19" extent="16-16"/>
+<wire x1="13" y1="18.85" x2="11.5" y2="17.2" width="0" layer="19" extent="16-16"/>
+<wire x1="24.25" y1="12.95" x2="20.75" y2="15.2" width="0" layer="19" extent="16-16"/>
 </signal>
 <signal name="INT0">
@@
 <contactref element="C5" pad="2"/>
 <contactref element="U$1" pad="28"/>
-<contactref element="R1" pad="1"/>
 <wire x1="12.9" y1="17.9" x2="12.9" y2="18.75" width="0.254" layer="16"/>
-<wire x1="12.9" y1="18.75" x2="13" y2="18.85" width="0.254" layer="16"/>
 <wire x1="24.9993" y1="24.5031" x2="24.9993" y2="25.2993" width="0.254" layer="16"/>
 <wire x1="24.9993" y1="25.2993" x2="25.2" y2="25.5" width="0.254" layer="16"/>
