File: schematics/v45/queso_dip_v4_5.brd (EAGLE design)
At the start: 41 x 50 mm, 49 parts, among them Q1 FOXSDLF/120-20, U1 PRTR5V0U2X,215, U2 PRTR5V0U2X,215, U3 PRTR5V0U2X,215, U4 PRTR5V0U2X,215, U5 PRTR5V0U2X,215, X1 USB-A-HU, X2 USB-A-HU, X3 USB-A-HU, X4 USB-A-HU

Commit message: sch + adapter
Routing:
- net N$3: track 3.65 -> 10.7 mm
- net N$4: track 3.09 -> 10.0 mm
- net N$5: track 3.17 -> 9.92 mm
- net N$1: track 3.71 -> 9.71 mm
- net GND: track 291.4 -> 293.6 mm
- net DM3: track 17.0 -> 18.4 mm
- net DP2: track 18.1 -> 19.5 mm
- net DM2: track 18.1 -> 19.4 mm
- net DM1: track 23.8 -> 25.1 mm
- net DP3: track 17.2 -> 18.3 mm
Other:
- board text added: "QUESO DIP II"
- board text added: "ordered 2016/04/13 elecrow"
- board text removed: "QUESO DIP"
- board text removed: "not ordered"
