File: schematics/v48/queso_dip_v4_8.sch (EAGLE design)
At the start: 50 parts, among them Q1 FOXSDLF/120-20, U1 PRTR5V0U2X,215, U2 PRTR5V0U2X,215, U3 PRTR5V0U2X,215, U4 PRTR5V0U2X,215, U5 PRTR5V0U2X,215, X1 USB-A-S, X2 USB-A-S, X3 USB-A-S, X4 USB-A-S

Commit message: fixed DRC
Parts:
- removed JP1: (no value), jumper:SJ2W
- removed USB1: USBUSB-MICROB-SMT-DIP, Spark:USBUSB-MICROB-SMT-DIP
- added POWER_USB: USBUSB-MICROB-SMT-DIP, Spark:USBUSB-MICROB-SMT-DIP
- added SJ3: (no value), SparkFun-Retired:SOLDERJUMPER_2WAYT
- X1, X2, X3, X4: value USB-A-S -> USB-A-HU; device con-usb:USB-A-S -> con-usb:USB-A-HU
- renumbered USB to DATA_USB
Connections:
- net DM1: now also X4.D+; no longer X4.D-
- net DM2: now also X3.D+; no longer X3.D-
- net DM3: now also X2.D+; no longer X2.D-
- net DM4: now also X1.D+; no longer X1.D-
- net DP1: now also X4.D-; no longer X4.D+
- net DP2: now also X3.D-; no longer X3.D+
- net DP3: now also X2.D-; no longer X2.D+
- net DP4: now also X1.D-; no longer X1.D+
- net GND: now also POWER_USB.GND, X1.VBUS, X2.VBUS, X3.VBUS, X4.VBUS; no longer USB1.GND, X1.GND, X2.GND, X3.GND, X4.GND
- net N$1: now also X1.GND; no longer X1.VBUS
- net N$3: now also X4.GND; no longer X4.VBUS
- net N$4: now also X2.GND; no longer X2.VBUS
- net N$5: now also X3.GND; no longer X3.VBUS
- net VCC: now also SJ3.2; no longer JP1.2
- net VIN: now also SJ3.1; no longer JP1.1
- net VOUT: now also POWER_USB.VBUS, SJ3.3; no longer JP1.3, USB1.VBUS
Other:
- moved on the sheet: D3
