File: schematics/v101/queso_dip_v101.brd (EAGLE design)
At the start: 41 x 50 mm, 51 parts, among them Q1 FOXSDLF/120-20, X1 USB-A-HU, X2 USB-A-HU, X3 USB-A-HU, X4 USB-A-HU

Commit message: added dual power
Parts:
- removed F1, F2, F3, F4: PTS12066V110, m-pad-2.1:1210
- added D2, D4: ES2D, diode:SMB
- C1, C2, C3, C4: value VJ1210V106ZXJTW1BC -> n.a.
- VD1, VD2, VD3: value USBLC6-4SC6 -> n.a.
- moved C6 6.17 mm to (9.90, 26.2)
- moved C12 2.65 mm to (11.9, 31.7)
- moved C13 2.65 mm to (15.2, 31.7)
- moved U$4 1.72 mm to (6.00, 35.2)
- moved R2 0.30 mm to (23.5, 34.9)
- moved R9 0.30 mm to (23.5, 37.2)
Connections:
- removed net N$3: F4.2, X4.VBUS
- removed net N$4: F1.2, X2.VBUS
- new net CHR: C12.2, C13.2, D2.A, L2.P$1, U$6.36
- net N$1: no longer F2.2, X1.VBUS
- net N$5: no longer F3.2, X3.VBUS
- net N$6: now also D4.A
- net VCC: now also D2.C, D4.C, X1.VBUS, X2.VBUS, X3.VBUS, X4.VBUS; no longer C12.2, C13.2, F1.1, F2.1, F3.1, F4.1, L2.P$1, U$6.36
Routing:
- net CHR: track 0.00 -> 28.2 mm
- net N$6: track 0.00 -> 28.0 mm
- net VCC: track 164.3 -> 184.9 mm
- net N$1: track 16.4 -> 5.38 mm
- net N$5: track 17.0 -> 6.08 mm
- net N$3: track 10.7 -> 0.00 mm
- net N$4: track 10.0 -> 0.00 mm
- net N$17: track 20.5 -> 24.6 mm
- net V_UP: track 38.6 -> 40.8 mm
- net N$11: track 8.72 -> 9.93 mm
- net GND: vias 7 -> 8
