File: schematics/v101/queso_dip_v101.sch (EAGLE design)
At the start: 51 parts, among them Q1 FOXSDLF/120-20, X1 USB-A-HU, X2 USB-A-HU, X3 USB-A-HU, X4 USB-A-HU

Commit message: added dual power
Parts:
- removed F1, F2, F3, F4: PTS12066V110, m-pad-2.1:FUSED
- added D2, D4: ES2D, diode:ES2D
- C1, C2, C3, C4: value VJ1210V106ZXJTW1BC -> n.a.
- VD1, VD2, VD3: value USBLC6-4SC6 -> n.a.
Connections:
- removed net N$3: F4.2, X4.GND
- removed net N$4: F1.2, X2.GND
- new net CHR: C12.2, C13.2, D2.A, L2.1, U$6.ACIN-5V
- net N$1: no longer F2.2, X1.GND
- net N$5: no longer F3.2, X3.GND
- net N$6: now also D4.A
- net VCC: now also D2.C, D4.C, X1.GND, X2.GND, X3.GND, X4.GND; no longer C12.2, C13.2, F1.1, F2.1, F3.1, F4.1, L2.1, U$6.ACIN-5V
